File: KiCAD/pid_controller/pid_controller.kicad_sch (KiCad schematic)
At the start: 39 parts, among them J1 12VDC Power In, J2 Heater, J4 Rotary Encoder, M1 Fan, Q1 irf3205/2SK3570/IPB11N03LA, Q2 N.A, Q3 irf3205/2SK3570/IPB11N03LA, Q4 N.A, U1 L7805, U2 LM35-LP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

Commit message: Redesign the PCB and add some other footprints
Parts:
- added D2: 1N4001, Diode_THT:D_DO-41_SOD81_P10.16mm_Horizontal, symbol Diode:1N4001
- added J3: +5V, Connector_PinHeader_2.54mm:PinHeader_2x02_P2.54mm_Vertical, symbol Connector_Generic:Conn_02x02_Counter_Clockwise
- added U6: 24LC64, Package_DIP:DIP-8_W10.16mm_LongPads, symbol Memory_EEPROM:24LC64
- M1: footprint (none) -> Connector_PinHeader_2.54mm:PinHeader_1x02_P2.54mm_Vertical
- R1, R11, R13, R15, R17, R18, R3, R5, R7, R9: footprint Resistor_SMD:R_1210_3225Metric_Pad1.42x2.65mm_HandSolder -> Resistor_SMD:R_1210_3225Metric
Connections:
- net +12V: now also D2.1 (K)
- net +5V: now also J3.1 (Pin_1), J3.2 (Pin_2), U6.8 (VCC)
- net GND: now also J3.3 (Pin_3), J3.4 (Pin_4), U6.1 (A0), U6.2 (A1), U6.4 (GND), U6.7 (WP)
- net SCL: now also U6.6 (SCL)
- net SDA: now also U6.5 (SDA)
- net at M1.2 (-), Q3.2 (D), Q4.2 (D): now also D2.2 (A)
- no-connect marks 17 -> 18
Other:
- note added: "N.A"
